File: hardware/orangecrab_r0.2.1/OrangeCrab.kicad_pcb (KiCad board)
At the start: 6 copper layers, 50.8 x 22.9 mm, 163 parts, among them J1 Conn_01x12_Male, J2 Conn_01x16_Male, J3 USB_C_Receptacle_USB2.0, J4 MicroSd, J5 JST, J6 Conn_01x05_Male, SW1 SW_Push, U1 TLV62569DRL, U10 NCP115-2.5, U2 TLV62569DRL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

Commit message: refresh
Routing:
- net RAM_D10: track 0.00 -> 4.20 mm
- net RAM_LDQS+: track 0.33 -> 4.18 mm
- net RAM_D9: track 2.10 -> 5.50 mm
- net RAM_D14: track 0.00 -> 3.00 mm
- net RAM_D11: track 1.39 -> 4.18 mm
- net RAM_LDQS-: track 0.92 -> 3.58 mm
- net GND: track 67.2 -> 69.4 mm
- net /DRAM/RAM_VDDQ: track 6.36 -> 8.17 mm
- net /DRAM/RAM_VDD: track 4.57 -> 6.16 mm
- net RAM_D12: track 0.00 -> 1.45 mm
- net RAM_D15: track 0.77 -> 1.76 mm

Commit message: refresh
Routing:
- net GND: track 69.4 -> 79.3 mm
- net RAM_A4: track 0.26 -> 4.50 mm
- net RAM_A1: track 0.86 -> 4.76 mm
- net RAM_A2: track 0.44 -> 3.87 mm
- net RAM_A6: track 0.00 -> 3.04 mm
- net RAM_A5: track 1.39 -> 4.22 mm
- net RAM_A11: track 0.86 -> 3.56 mm
- net /DRAM/RAM_VDD: track 6.16 -> 8.43 mm
- net RAM_A9: track 0.71 -> 2.94 mm
- net RAM_A8: track 0.27 -> 2.11 mm
- net RAM_A7: track 2.25 -> 3.88 mm
- net RAM_A14: track 0.26 -> 1.75 mm
- net RAM_D5: track 0.85 -> 2.26 mm
- net /DRAM/RAM_ZQ: track 0.00 -> 1.41 mm
- net RAM_D3: track 0.00 -> 1.41 mm
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