File: hardware/orangecrab_r0.2.1/OrangeCrab.kicad_pcb (KiCad board)
At the start: 6 copper layers, 50.8 x 22.9 mm, 163 parts, among them J1 Conn_01x12_Male, J2 Conn_01x16_Male, J3 USB_C_Receptacle_USB2.0, J4 MicroSd, J5 JST, J6 Conn_01x05_Male, SW1 SW_Push, U1 TLV62569DRL, U10 NCP115-2.5, U2 TLV62569DRL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

Commit message: refresh
Routing:
- net /DRAM/RAM_VDD: track 8.43 -> 22.3 mm, vias 0 -> 4
- net ECP5_VREF: track 5.94 -> 15.4 mm, vias 0 -> 2
- net /DRAM/RAM_VDDQ: track 8.17 -> 16.6 mm
- net (no net): track 1.79 -> 6.52 mm, vias 0 -> 2
- net GND: track 79.3 -> 80.1 mm

Commit message: refresh
Parts:
- moved G*** 0.69 mm to (181.5, 102.6)
Routing:
- net GND: track 80.1 -> 89.3 mm
- net /DRAM/RAM_VDDQ: track 16.6 -> 22.8 mm, vias 0 -> 1
- net /DRAM/RAM_VDD: track 22.3 -> 27.9 mm, vias 4 -> 5
- net ECP5_VREF: track 15.4 -> 16.0 mm
